File: hardware/prj-kicad/cowdin-3c-esp-ui.kicad_sch (KiCad schematic)
At the start: 18 parts, among them P1 CONN_F52R-04, SW1 SW_PUSH, SW2 SW_PUSH, SW3 SW_PUSH, SW4 SW_PUSH, SW5 SW_PUSH

Commit message: Hardware: Add MCU and main components. Create productions files for rev1
Parts:
- added C11, C12, C13: 1uF, cowdin-3c-esp-ui:SMD0603, symbol cowdin-3c-esp-ui:C
- added C14, C15, C17, C18: 100nF, cowdin-3c-esp-ui:SMD0603, symbol cowdin-3c-esp-ui:C
- added C16: 4,7uF, cowdin-3c-esp-ui:SMD0805, symbol cowdin-3c-esp-ui:C
- added D1: USBLC6-2, cowdin-3c-esp-ui:SOT23-6, symbol cowdin-3c-esp-ui:USBLC6-2
- added D2: LED, cowdin-3c-esp-ui:SMD0805, symbol cowdin-3c-esp-ui:LED
- added P2: CONN_TC2030, cowdin-3c-esp-ui:TC2030-MCP-FP, symbol cowdin-3c-esp-ui:CONN_TC2030
- added R2: 10k, cowdin-3c-esp-ui:SMD0603, symbol cowdin-3c-esp-ui:R
- added R3: 330, cowdin-3c-esp-ui:SMD0603, symbol cowdin-3c-esp-ui:R
- added SHLD1, SHLD2, SHLD3, SHLD4: CONN_1, cowdin-3c-esp-ui:SHLD_PAD, symbol cowdin-3c-esp-ui:CONN_1
- added TP1, TP2, TP3: CONN_1, cowdin-3c-esp-ui:TP_SMD, symbol cowdin-3c-esp-ui:CONN_1
- added U1: ATSAMD21Exx, cowdin-3c-esp-ui:TQFP32, symbol cowdin-3c-esp-ui:ATSAMD21Exx
- added U2: W25Q16JV, cowdin-3c-esp-ui:SOIC-8, symbol cowdin-3c-esp-ui:W25Q16JV
Connections:
- net +3.3V: now also DISP1.6 (VBAT), DISP1.9 (VDD), C14.1, C15.1, C16.1, C17.1, C18.1, R2.1, R3.1, U1.30 (VDD), U1.9 (ANA), U2.3 (IO2_WP), U2.7 (IO3_HOLD), U2.8
- net GND: now also DISP1.10 (BS0), DISP1.11 (BS1), DISP1.12 (BS2), C11.2, C12.2, C13.2, C14.2, C15.2, C16.2, C17.2, C18.2, D1.2, P2.5 (GND), SHLD1.1, SHLD2.1, SHLD3.1, SHLD4.1, TP3.1, U1.10, U1.28, U2.4
- net SW1: now also U1.25 (PA27)
- net SW2: now also U1.14 (PA11)
- net SW3: now also U1.15 (PA14)
- net SW4: now also U1.13 (PA10)
- net SW5: now also U1.16 (PA15)
- net UART_RX: now reaches P1.2 (PM)
- net UART_RX: now also U1.22 (PA23)
- net UART_TX: now reaches P1.3 (P3)
- net UART_TX: now also U1.21 (PA22)
- net DISP_SCS: now reaches DISP1.13 (CS)
- net DISP_SCS: now also U1.7 (PA06)
- net DISP_RST: now reaches DISP1.14 (RES)
- net DISP_RST: now also U1.4 (PA03)
- net DISP_DC: now reaches DISP1.15 (D/C)
- net DISP_DC: now also U1.3 (PA02)
- net DISP_RW: now reaches DISP1.16 (RW)
- net DISP_RW: now also U1.2 (PA01)
- net DISP_ERD: now reaches DISP1.17 (E/RD)
- net DISP_ERD: now also U1.1 (PA00)
- net DISP_SCK: now reaches DISP1.18 (D0)
- net DISP_SCK: now also U1.6 (PA05)
- net DISP_MOSI: now reaches DISP1.19 (D1)
- net DISP_MOSI: now also U1.5 (PA04)
- new net: D2.1 (A), R3.2
- new net: D1.1 (IO1), P2.3 (USB1)
- new net: D1.3 (IO2), P2.4 (USB2)
- new net: TP1.1, U1.11 (PA08)
- new net: TP2.1, U1.12 (PA09)
- new net +VCORE: C12.1, U1.29 (CORE)
- new net +VUSB: C11.1, D1.5, P2.1 (PWR)
- new net DISP_MISO: U1.8 (PA07)
- new net LED1: D2.2 (K), U1.27 (PA28)
- new net MEM_MISO: U1.20 (PA19), U2.2 (IO1_DO)
- new net MEM_MOSI: U1.17 (PA16), U2.5 (IO0_DI)
- new net MEM_SCK: U1.18 (PA17), U2.6 (CLK)
- new net MEM_SCS: U1.19 (PA18), U2.1 (CS)
- new net RST: C13.1, R2.2, U1.26 (RST)
- new net SWCLK: P2.6 (DBG2), U1.31 (PA30)
- new net SWDAT: P2.2 (DBG1), U1.32 (PA31)
- new net USB_D+: D1.4 (IO2), U1.24 (PA25)
- new net USB_D-: D1.6 (IO1), U1.23 (PA24)
- no-connect marks 8 -> 6
Other:
- moved on the sheet: C10, C2, C3, C4, C5, C6, C7, C8, C9, R1, SW1, SW2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
